File: analog-amplifier/analog-amplifier.kicad_sch (KiCad schematic)
At the start: 0 parts

Commit message: Prototype schematics
Parts:
- added C1, C10, C11, C12, C13, C9: 100n, Capacitor_SMD:C_0603_1608Metric, symbol Device:C
- added C2, C5: 10n, Capacitor_SMD:C_0603_1608Metric, symbol Device:C
- added C3, C4, C6, C7: 1.5p, Capacitor_SMD:C_0603_1608Metric, symbol Device:C
- added C8: 1u, Capacitor_SMD:C_0805_2012Metric, symbol Device:C
- added J1, J2, J3, J4: Conn_Coaxial_Small, Connector_Coaxial:SMA_Amphenol_132289_EdgeMount, symbol Connector:Conn_Coaxial_Small
- added JP1, JP2: Jumper_2_Open, TestPoint:TestPoint_2Pads_Pitch2.54mm_Drill0.8mm, symbol Jumper:Jumper_2_Open
- added R1: 1.2k, Resistor_SMD:R_0603_1608Metric, symbol Device:R
- added R10, R11, R12, R5: 49.9, Resistor_SMD:R_0603_1608Metric, symbol Device:R
- added R13, R14: 499, Resistor_SMD:R_0603_1608Metric, symbol Device:R
- added R2: 2.2k, Resistor_SMD:R_0603_1608Metric, symbol Device:R
- added R3, R8: 2.5Meg, Resistor_SMD:R_0603_1608Metric, symbol Device:R
- added R4, R9: 1Meg, Resistor_SMD:R_0603_1608Metric, symbol Device:R
- added R6, R7: 1k, Resistor_SMD:R_0603_1608Metric, symbol Device:R
- added U1, U3: LT6202, Package_SO:SO-8_3.9x4.9mm_P1.27mm, symbol LT6202:LT6202
- added U2, U4: LT6404IUD, Package_DFN_QFN:QFN-16-1EP_3x3mm_P0.5mm_EP1.45x1.45mm, symbol LTC6404IUD:LT6404IUD
Connections:
- new net: C6.2, R11.2, R13.1, U4.15 (IN+)
- new net: C6.1, R13.2, U4.14 (OUT-)
- new net: C3.1, R11.1, R6.2, U2.14 (OUT-)
- new net: R10.1, U3.2 (IN-), U3.6 (OUT)
- new net: C5.2, JP2.2 (B), R8.2, R9.1, U3.3 (IN+)
- new net: C3.2, R5.2, R6.1, U2.15 (IN+)
- new net: C4.1, R10.2, R7.2, U2.6 (IN-)
- new net: C7.1, R12.2, R14.2, U4.6 (IN-)
- new net: C7.2, R14.1, U4.7 (OUT+)
- new net: R5.1, U1.2 (IN-), U1.6 (OUT)
- new net: C2.2, JP1.2 (B), R3.2, R4.1, U1.3 (IN+)
- new net: C4.2, R12.1, R7.1, U2.7 (OUT+)
- new net +3V0: C1.1, R1.2, R2.1, U2.4 (Vocm), U4.4 (Vocm)
- new net +5V: C10.1, C11.1, C12.1, C13.1, C8.1, C9.1, R1.1, R3.1, R8.1, U1.7 (V+), U2.1 (nSHDN), U2.10 (V+), U2.11 (V+), U2.2 (V+), U3.7 (V+), U4.1 (nSHDN), U4.10 (V+), U4.11 (V+), U4.2 (V+)
- new net GND: C1.2, C10.2, C11.2, C12.2, C13.2, C8.2, C9.2, J1.2 (Ext), J2.2 (Ext), J3.2 (Ext), J4.2 (Ext), R2.2, R4.2, R9.2, U1.4 (V-), U2.12 (V-), U2.17 (PAD), U2.3 (V-), U2.9 (V-), U3.4 (V-), U4.12 (V-), U4.17 (PAD), U4.3 (V-), U4.9 (V-)
- new net IN+: C2.1, J1.1 (In), JP1.1 (A)
- new net IN-: C5.1, J2.1 (In), JP2.1 (A)
- new net OUT+: J4.1 (In), U4.8 (OUTF+)
- new net OUT-: J3.1 (In), U4.13 (OUTF-)
- no-connect marks 0 -> 2
Other:
- note added: "As near to +V pin as possible"
- note added: "LT6202 supply filter"
- note added: "Power supply"
- note added: "Power supply filter"
- note added: "k=10"
- note added: "k=20"

Commit message: Draft of the layout
Parts:
- removed R1: 1.2k, Resistor_SMD:R_0603_1608Metric, symbol Device:R
- added C14, C15, C16, C17: 100n, Capacitor_SMD:C_0603_1608Metric, symbol Device:C
- added D1: D_Zener 5.1V, Package_TO_SOT_SMD:SOT-23-3, symbol Device:D_Zener
- added D2: SS14, Diode_SMD:D_SMA, symbol Diode:SS14
- added F1: Polyfuse, Resistor_SMD:R_0603_1608Metric, symbol Device:Polyfuse
- added J5, J6: Conn_01x01_Socket, Connector_PinSocket_2.54mm:PinSocket_1x01_P2.54mm_Vertical, symbol Connector:Conn_01x01_Socket
- added JP3, JP4: Jumper_2_Open, Connector_PinSocket_1.27mm:PinSocket_1x02_P1.27mm_Vertical, symbol Jumper:Jumper_2_Open
- added R15: 28k, Resistor_SMD:R_0603_1608Metric, symbol Device:R
- JP1, JP2: footprint TestPoint:TestPoint_2Pads_Pitch2.54mm_Drill0.8mm -> Connector_PinSocket_2.54mm:PinSocket_1x02_P2.54mm_Vertical
- R2: value 2.2k -> 28k
- U1, U3: LCSC (none) -> C672942
Connections:
- net +5V: now also C1.1, R2.2, C15.1, C16.1, C17.1, D1.1 (K), D2.1 (K), F1.2, R15.2; no longer C9.1
- net GND: now also C9.1, C14.1, C15.2, C16.2, C17.2, D1.2 (A), D2.2 (A), J6.1 (Pin_1); no longer C9.2, R2.2
- net IN+: now also JP3.2 (B)
- net IN-: now also JP4.2 (B)
- net at C5.2, JP2.2 (B), R8.2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: now also JP4.1 (A)
- net at C2.2, JP1.2 (B), R3.2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: now also JP3.1 (A)
- net +3V0: no longer names the net of R2.1, U4.4 (Vocm)
- net +3V0: now also C9.2; no longer C1.1, U2.4 (Vocm)
- new net: F1.1, J5.1 (Pin_1)
- new net: C14.2, R15.1, U2.4 (Vocm)
Other:
- note added: "Circuit protection and power supply"
- note added: "LTC6404 filters"
- note removed: "Power supply"
- note removed: "Power supply filter"
- moved on the sheet: C10, C11, C12, C13, R10

Commit message: Finished Beta
Parts:
- removed JP3, JP4: Jumper_2_Open, Connector_PinSocket_1.27mm:PinSocket_1x02_P1.27mm_Vertical, symbol Jumper:Jumper_2_Open
- J1, J2, J3, J4: footprint Connector_Coaxial:SMA_Amphenol_132289_EdgeMount -> Connector_Coaxial:SMA_Samtec_SMA-J-P-X-ST-EM1_EdgeMount
Changed lines of the file:
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@@
-    (stroke (width 0) (type default))
-  )
-  (wire (pts (xy 49.53 93.98) (xy 49.53 104.14))
     (stroke (width 0) (type default))
   )
@@
     (stroke (width 0) (type default))
   )
-  (wire (pts (xy 59.69 138.43) (xy 59.69 148.59))
-    (stroke (width 0) (type default))
-  )
   (wire (pts (xy 224.79 124.46) (xy 224.79 129.54))
     (stroke (width 0) (type default))
@@
     (stroke (width 0) (type default))
   )
-  (wire (pts (xy 49.53 138.43) (xy 49.53 148.59))
-    (stroke (width 0) (type default))
-  )
   (wire (pts (xy 153.67 124.46) (xy 153.67 130.81))
     (stroke (width 0) (type default))
@@
   )
   (wire (pts (xy 242.57 120.65) (xy 242.57 123.19))
-    (stroke (width 0) (type default))
-  )
-  (wire (pts (xy 59.69 93.98) (xy 59.69 104.14))
     (stroke (width 0) (type default))
   )
@@
   (label "IN-" (at 43.18 138.43 180) (fields_autoplaced)
     (effects (font (size 1.27 1.27)) (justify right bottom))
-  )
-  (symbol (lib_id "Jumper:Jumper_2_Open") (at 54.61 104.14 0) (mirror y) (unit 1)
-    (in_bom yes) (on_board yes) (dnp no)
-    (property "Reference" "JP3" (at 54.61 109.22 0)
-      (effects (font (size 1.27 1.27)))
-    )
-    (property "Value" "Jumper_2_Open" (at 54.61 106.68 0)
-      (effects (font (size 1.27 1.27)))
-    )
-    (property "Footprint" "Connector_PinSocket_1.27mm:PinSocket_1x02_P1.27mm_Vertical" (at 54.61 104.14 0)
-      (effects (font (size 1.27 1.27)) hide)
-    )
-    (property "Datasheet" "~" (at 54.61 104.14 0)
-      (effects (font (size 1.27 1.27)) hide)
-    )
-    (pin "1")
-    (pin "2")
-    (instances
-      (project "analog-amplifier"
-        (path "/ce61e0ad-f414-485d-bc43-268c32387575"
-          (reference "JP3") (unit 1)
-        )
-      )
-    )
   )
   (symbol (lib_id "power:+5V") (at 195.58 106.68 0) (unit 1)
@@
       (effects (font (size 1.27 1.27)))
     )
-    (property "Footprint" "Connector_Coaxial:SMA_Amphenol_132289_EdgeMount" (at 261.62 129.54 0)
+    (property "Footprint" "Connector_Coaxial:SMA_Samtec_SMA-J-P-X-ST-EM1_EdgeMount" (at 261.62 129.54 0)
       (effects (font (size 1.27 1.27)) hide)
     )
@@
       (effects (font (size 1.27 1.27)))
     )
-    (property "Footprint" "Connector_Coaxial:SMA_Amphenol_132289_EdgeMount" (at 21.59 93.98 0)
+    (property "Footprint" "Connector_Coaxial:SMA_Samtec_SMA-J-P-X-ST-EM1_EdgeMount" (at 21.59 93.98 0)
       (effects (font (size 1.27 1.27)) hide)
     )
@@
       (effects (font (size 1.27 1.27)))
     )
-    (property "Footprint" "Connector_Coaxial:SMA_Amphenol_132289_EdgeMount" (at 21.59 138.43 0)
+    (property "Footprint" "Connector_Coaxial:SMA_Samtec_SMA-J-P-X-ST-EM1_EdgeMount" (at 21.59 138.43 0)
       (effects (font (size 1.27 1.27)) hide)
     )
@@
         (path "/ce61e0ad-f414-485d-bc43-268c32387575"
           (reference "#PWR011") (unit 1)
-        )
-      )
-    )
-  )
-  (symbol (lib_id "Jumper:Jumper_2_Open") (at 54.61 148.59 0) (mirror y) (unit 1)
-    (in_bom yes) (on_board yes) (dnp no)
-    (property "Reference" "JP4" (at 54.61 153.67 0)
-      (effects (font (size 1.27 1.27)))
-    )
-    (property "Value" "Jumper_2_Open" (at 54.61 151.13 0)
-      (effects (font (size 1.27 1.27)))
-    )
-    (property "Footprint" "Connector_PinSocket_1.27mm:PinSocket_1x02_P1.27mm_Vertical" (at 54.61 148.59 0)
-      (effects (font (size 1.27 1.27)) hide)
-    )
-    (property "Datasheet" "~" (at 54.61 148.59 0)
-      (effects (font (size 1.27 1.27)) hide)
-    )
-    (pin "1")
-    (pin "2")
-    (instances
-      (project "analog-amplifier"
-        (path "/ce61e0ad-f414-485d-bc43-268c32387575"
-          (reference "JP4") (unit 1)
         )
       )
@@
       (effects (font (size 1.27 1.27)))
     )
-    (property "Footprint" "Connector_Coaxial:SMA_Amphenol_132289_EdgeMount" (at 261.62 97.79 0)
-      (effects (font (size 1.27 1.27)) hide)
-    )
+    (property "Footprint" "Connector_Coaxial:SMA_Samtec_SMA-J-P-X-ST-EM1_EdgeMount" (at 261.62 97.79 0)
+      (effects (font (size 1.27 1.27)) hide)
+    )

Commit message: Added gerbers
Parts:
- R10, R11, R12, R5: LCSC (none) -> C23185
- R6, R7: LCSC (none) -> C21190
Changed lines of the file:
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@@
+      (effects (font (size 1.27 1.27)) hide)
+    )
+    (property "LCSC" "C23185" (at 193.04 91.44 90)
       (effects (font (size 1.27 1.27)) hide)
     )
@@
       (effects (font (size 1.27 1.27)) hide)
     )
+    (property "LCSC" "C21190" (at 152.4 91.44 90)
+      (effects (font (size 1.27 1.27)) hide)
+    )
     (pin "2")
     (pin "1")
@@
     )
     (property "Datasheet" "~" (at 124.46 135.89 0)
+      (effects (font (size 1.27 1.27)) hide)
+    )
+    (property "LCSC" "C23185" (at 124.46 135.89 90)
       (effects (font (size 1.27 1.27)) hide)
     )
@@
       (effects (font (size 1.27 1.27)) hide)
     )
+    (property "LCSC" "C21190" (at 152.4 135.89 90)
+      (effects (font (size 1.27 1.27)) hide)
+    )
     (pin "2")
     (pin "1")
@@
     )
     (property "Datasheet" "~" (at 133.35 91.44 0)
+      (effects (font (size 1.27 1.27)) hide)
+    )
+    (property "LCSC" "C23185" (at 133.35 91.44 90)
       (effects (font (size 1.27 1.27)) hide)
     )
@@
       (effects (font (size 1.27 1.27)) hide)
     )
+    (property "LCSC" "C23185" (at 193.04 135.89 90)
+      (effects (font (size 1.27 1.27)) hide)
+    )
